File: atmega328.kicad_pcb (KiCad board)
At the start: 2 copper layers, 82 parts, among them J1 JST-XH 3-pin, J2 USB_C_Receptacle_USB2.0_16P, J3 Conn_Coaxial, J4 Video_Out, J5 AVR ICSP, J6 Conn_01x01, J7 Conn_01x01, J8 Conn_01x01, J9 Conn_01x01, Q1 AO3400A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

Commit message: fixed positions
Parts:
- moved R1 39.8 mm to (174.0, 136.2), turned to 90 degrees
- moved U2 38.0 mm to (179.0, 133.1)
- moved R14 37.9 mm to (159.4, 131.8)
- moved C14 37.8 mm to (153.5, 117.0), turned to 90 degrees
- moved R2 37.7 mm to (179.2, 137.9)
- moved C34 37.3 mm to (184.0, 137.5)
- moved C16 37.1 mm to (153.2, 106.0)
- moved L2 34.9 mm to (192.0, 128.0), turned to -90 degrees
- moved R13 33.8 mm to (159.3, 134.0)
- moved R7 32.8 mm to (153.5, 120.8)
- moved C33 32.8 mm to (183.0, 127.2)
- moved L1 31.7 mm to (167.2, 105.0)
- moved Q3 31.4 mm to (162.9, 110.0)
- moved J1 31.4 mm to (168.8, 141.7), turned to -90 degrees
- moved Q1 30.9 mm to (158.3, 110.0)
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Routing:
- added copper zone on B.Cu, net GND
- added copper zone on F.Cu, net GND
Other:
- board outline added: 114.2 x 102.8 mm

Commit message: fixed positions 2
Parts:
- moved L1 5.00 mm to (172.2, 105.0)
- moved L2 1.90 mm to (190.2, 127.2)
Changed lines of the file:
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@@
 	(footprint "Inductor_THT:L_Radial_D10.0mm_P5.00mm_Fastron_07M"
 		(layer "F.Cu")
-		(at 167.25 105)
+		(at 172.25 105)
 		(descr "Inductor, Radial series, Radial, pin pitch=5.00mm, diameter=10mm, height=12.7mm, Fastron, 07M, http://www.fastrongroup.com/image-show/37/07M.pdf?type=Complete-DataSheet&productType=series")
 		(tags "Inductor Radial series Radial pin pitch 5.00mm  diameter 10mm height 12.7mm Fastron 07M")
@@
 	(footprint "Inductor_THT:L_Radial_D10.0mm_P5.00mm_Fastron_07M"
 		(layer "F.Cu")
-		(at 192 128 -90)
+		(at 190.25 127.25 -90)
 		(descr "Inductor, Radial series, Radial, pin pitch=5.00mm, diameter=10mm, height=12.7mm, Fastron, 07M, http://www.fastrongroup.com/image-show/37/07M.pdf?type=Complete-DataSheet&productType=series")
 		(tags "Inductor Radial series Radial pin pitch 5.00mm  diameter 10mm height 12.7mm Fastron 07M")
@@
 		(min_thickness 0.25)
 		(filled_areas_thickness no)
-		(fill yes
+		(fill
 			(thermal_gap 0.5)
 			(thermal_bridge_width 0.5)
@@
 		(min_thickness 0.25)
 		(filled_areas_thickness no)
-		(fill yes
+		(fill
 			(thermal_gap 0.5)
 			(thermal_bridge_width 0.5)
@@
 		(polygon
 			(pts
-				(xy 86.75 58.5) (xy 86.75 58.5) (xy 201 58.5) (xy 201 161.25) (xy 86.75 161.25)
+				(xy 86.75 58.5) (xy 201 58.5) (xy 201 161.25) (xy 86.75 161.25)
 			)
 		)

Commit message: fixed all errors and warnings
Parts:
- moved Q6 43.6 mm to (120.2, 158.4), turned to -90 degrees
- moved Q7 39.9 mm to (118.1, 152.9), turned to 180 degrees
- moved U1 39.0 mm to (124.8, 154.4)
- moved R9 38.9 mm to (118.9, 149.5)
- moved R1 38.6 mm to (141.5, 157.1)
- moved C34 37.6 mm to (151.0, 155.5)
- moved L2 37.3 mm to (160.0, 149.0)
- moved R2 36.7 mm to (146.9, 155.5)
- moved J2 36.6 mm to (97.7, 158.4)
- moved U2 35.1 mm to (147.5, 148.5)
- moved U6 34.8 mm to (104.8, 142.4), turned to 90 degrees
- moved J1 34.3 mm to (136.0, 152.0)
- moved C32 33.1 mm to (100.0, 148.0)
- moved C17 32.5 mm to (129.5, 149.5)
- moved J8 30.8 mm to (89.5, 141.5)
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Other:
- board size 114.2 x 102.8 mm -> 80.8 x 102.8 mm

Commit message: added connections
Parts:
- moved R4 11.7 mm to (95.6, 152.0), turned to 0 degrees
- moved Y2 10.9 mm to (113.7, 113.9)
- moved C29 10.3 mm to (118.5, 119.5), turned to 0 degrees
- moved R5 10.0 mm to (102.9, 151.0)
- moved C30 5.59 mm to (118.5, 114.0)
- moved C15 5.00 mm to (143.0, 119.5), turned to 0 degrees
- moved R7 4.58 mm to (126.5, 127.5)
- moved R18 4.00 mm to (103.0, 133.0), turned to 180 degrees
- moved C14 3.81 mm to (133.5, 110.5), turned to 0 degrees
- moved R11 2.66 mm to (129.5, 113.0)
- moved C32 2.12 mm to (98.5, 146.5)
- moved F1 1.50 mm to (107.5, 150.5), turned to 0 degrees
- moved C21 1.00 mm to (144.0, 62.3)
- moved Q2 0.63 mm to (148.5, 123.5), turned to 180 degrees
- moved R8 0.07 mm to (147.0, 133.0)
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Routing:
- net VSYS: track 0.00 -> 180.6 mm
- net VBUS_FUSED: track 0.00 -> 114.6 mm
- net GND: track 0.00 -> 93.0 mm, vias 0 -> 62
- net MCU_SDA: track 0.00 -> 77.9 mm, vias 0 -> 2
- net Net-(J5-Pin_5): track 0.00 -> 76.9 mm
- net RSSI_ADC: track 0.00 -> 67.5 mm, vias 0 -> 1
- net /MCU_Block/DTR: track 0.00 -> 66.6 mm, vias 0 -> 1
- net MCU_SCL: track 0.00 -> 60.2 mm, vias 0 -> 2
- net Net-(U3-ILIM_HIZ): track 0.00 -> 59.0 mm
- net VBAT: track 0.00 -> 58.0 mm
- net /Power_Block/REGN: track 0.00 -> 57.4 mm
- net SPI_SCK: track 0.00 -> 56.0 mm
- net D_MINUS: track 0.00 -> 54.6 mm
- net Net-(U6-VDD): track 0.00 -> 54.3 mm
- net SPI_MOSI: track 0.00 -> 50.6 mm, vias 0 -> 2
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- added copper zone on In2.Cu, net +3.3V
- added copper zone on In1.Cu, net GND
Other:
- board size 80.8 x 102.8 mm -> 80.8 x 102.2 mm
- copper layers 2 -> 4

Commit message: fixed positions of connections
Routing:
- net VBUS_FUSED: track 114.6 -> 125.5 mm
- net D_MINUS: track 54.6 -> 47.4 mm
- net /MCU_Block/DTR: track 66.6 -> 61.2 mm
- net Net-(U6-VDD): track 54.3 -> 49.0 mm
- net VBAT: track 58.0 -> 53.0 mm
- net Net-(F1-Pad1): track 19.9 -> 15.8 mm
- net /Power_Block/SRP: track 19.6 -> 16.4 mm
- net /Power_Block/VBAT-: track 24.3 -> 22.1 mm
- net Net-(Q2-G): track 20.2 -> 18.1 mm
- net D_PLUS: track 19.5 -> 17.6 mm
- net Net-(J5-Pin_5): track 76.9 -> 78.5 mm
- net Net-(U2-SW): track 11.9 -> 10.6 mm
- net /MCU_Block/PC3: track 24.3 -> 23.4 mm
- net /Power_Block/ACN: track 49.4 -> 48.9 mm
Other:
- board size 80.8 x 102.2 mm -> 80.7 x 102.7 mm
