File: atmega328.kicad_pcb (KiCad board)
At the start: 4 copper layers, 80.7 x 102.7 mm, 82 parts, among them J1 JST-XH 3-pin, J2 USB_C_Receptacle_USB2.0_16P, J3 Conn_Coaxial, J4 Video_Out, J5 AVR ICSP, J6 Conn_01x01, J7 Conn_01x01, J8 Conn_01x01, J9 Conn_01x01, Q1 AO3400A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

Commit message: Force update local files
Parts:
- added H1: MountingHole, MountingHole:MountingHole_3.2mm_M3, F.Cu at (163.9, 62.0)
- added H2: MountingHole, MountingHole:MountingHole_3.2mm_M3, F.Cu at (163.9, 157.6)
- added H3: MountingHole, MountingHole:MountingHole_3.2mm_M3, F.Cu at (90.3, 62.1)
- added H4: MountingHole, MountingHole:MountingHole_3.2mm_M3, F.Cu at (90.3, 157.7)
- added PC3 atmega: Conn_01x01, Connector_PinHeader_2.54mm:PinHeader_1x01_P2.54mm_Vertical, F.Cu at (89.4, 147.6)
- C1, C11, C14, C15, C17, C18, C19, C2, C20, C22, C23, C25, C27, C28, C29, C3, C30, C31, C32, C8, CУ1: footprint Capacitor_THT:C_Disc_D5.0mm_W2.5mm_P5.00mm -> Capacitor_SMD:C_0805_2012Metric
- C10, C16, C26, C33, C34, C9: footprint Capacitor_THT:CP_Radial_D5.0mm_P2.00mm -> Capacitor_SMD:CP_Elec_5x5.4
- C21: footprint Capacitor_THT:CP_Radial_D8.0mm_P3.50mm -> Capacitor_SMD:CP_Elec_8x10
- D1: footprint LED_THT:LED_D5.0mm -> LED_SMD:LED_0805_2012Metric
- L1, L2: footprint Inductor_THT:L_Radial_D10.0mm_P5.00mm_Fastron_07M -> Inductor_SMD:L_10.4x10.4_H4.8
- SW1, SW2, SW3: footprint Button_Switch_THT:SW_PUSH_6mm -> Button_Switch_SMD:SW_SPST_PTS645Sx43SMTR92
- moved J9 7.65 mm to (96.3, 134.2)
- moved C33 7.60 mm to (157.0, 134.4)
- moved C21 6.06 mm to (149.8, 64.1), turned to 0 degrees
- moved FB3 5.55 mm to (93.8, 115.9), turned to 180 degrees
- moved R23 4.47 mm to (93.3, 102.4)
- moved J2 4.37 mm to (102.0, 158.4)
- moved R4 4.23 mm to (99.0, 149.5), turned to 90 degrees
- moved R15 3.86 mm to (96.2, 138.1), turned to 90 degrees
- moved L2 3.76 mm to (160.2, 145.2)
- moved C26 3.65 mm to (139.9, 72.7)
- moved C15 2.92 mm to (145.5, 118.0)
- moved C34 2.75 mm to (153.8, 155.7)
- moved C1 2.64 mm to (131.6, 105.7)
- moved J3 2.23 mm to (90.2, 87.2)
- moved R18 2.10 mm to (103.1, 135.1)
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- renumbered U4 to RX5808
Connections:
- J9 pad 1: /MCU_Block/PC3 -> Net-(J9-Pin_1)
- R15 pad 2: /MCU_Block/PC3 -> Net-(J9-Pin_1)
Routing:
- net VBUS_FUSED: track 125.5 -> 66.3 mm, vias 0 -> 2
- net Net-(U3-ILIM_HIZ): track 59.0 -> 10.5 mm
- net Net-(U6-VDD): track 49.0 -> 3.12 mm
- net /MCU_Block/DTR: track 61.2 -> 95.4 mm, vias 1 -> 2
- net Net-(U3-BTST1): track 43.3 -> 10.2 mm
- net SPI_MOSI: track 51.0 -> 81.7 mm, vias 2 -> 0
- net D_MINUS: track 47.4 -> 17.1 mm
- net SPI_CS: track 42.3 -> 70.6 mm
- net SPI_MISO: track 44.3 -> 71.3 mm, vias 1 -> 2
- net SPI_SCK: track 56.0 -> 82.6 mm, vias 0 -> 2
- net VSYS: track 180.3 -> 155.5 mm, vias 0 -> 2
- net Net-(J5-Pin_5): track 78.5 -> 101.5 mm, vias 0 -> 1
- net GND: track 93.0 -> 115.9 mm, vias 62 -> 57
- net /Power_Block/REGN: track 57.8 -> 36.7 mm, vias 0 -> 2
- net MCU_SDA: track 77.9 -> 59.5 mm
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
Commit message: done with lcsc
Parts:
- C10, C16, C26, C33, C34, C9: footprint Capacitor_SMD:CP_Elec_5x5.4 -> Capacitor_SMD:C_0805_2012Metric
- FB3: value FerriteBead -> 600Ω @ 100MHz
- J10: renamed from PC3 atmega
- L1: value L -> 2.2µH
- renumbered RX5808 to U4
Routing:
- net VBUS_FUSED: track 66.3 -> 69.8 mm
- net VSYS: track 155.5 -> 156.8 mm
- net +3.3V: track 33.3 -> 34.6 mm
- net GND: track 115.9 -> 115.0 mm
- net Net-(U4-Vcc): track 27.4 -> 28.0 mm
- net /Power_Block/REGN: track 36.7 -> 36.1 mm
