File: atmega328.kicad_pcb (KiCad board)
At the start: 4 copper layers, 80.7 x 102.7 mm, 87 parts, among them J1 JST-XH 3-pin, J10 Conn_01x01, J2 USB_C_Receptacle_USB2.0_16P, J3 Conn_Coaxial, J4 Video_Out, J5 AVR ICSP, J6 Conn_01x01, J7 Conn_01x01, J8 Conn_01x01, J9 Conn_01x01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

Commit message: .
Routing:
- net GND: track 115.0 -> 116.3 mm
Changed lines of the file:
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@@
+	)
+	(segment
+		(start 112.5 152.405113)
+		(end 112.5 155.5)
+		(width 0.5)
+		(layer "F.Cu")
+		(net "GND")
 	)
 	(segment
@@
 		(width 0.5)
 		(layer "F.Cu")
-		(net "GND")
-	)
-	(segment
-		(start 112.5 153.655113)
-		(end 112.5 155.5)
-		(width 0.5)
-		(layer "F.Cu")
