File: _autosave-atmega328.kicad_pcb (KiCad board)
At the start: 4 copper layers, 80.7 x 102.7 mm, 87 parts, among them J1 JST-XH 3-pin, J10 Conn_01x01, J2 USB_C_Receptacle_USB2.0_16P, J3 Conn_Coaxial, J4 Video_Out, J5 AVR ICSP, J6 Conn_01x01, J7 Conn_01x01, J8 Conn_01x01, J9 Conn_01x01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

Commit message: production
Parts:
- renumbered CУ1 to CU1
Changed lines of the file:
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@@
 		(descr "Capacitor SMD 0805 (2012 Metric), square (rectangular) end terminal, IPC-7351 nominal, (Body size source: IPC-SM-782 page 76, https://www.pcb-3d.com/wordpress/wp-content/uploads/ipc-sm-782a_amendment_1_and_2.pdf, https://docs.google.com/spreadsheets/d/1BsfQQcO9C6DZCsRaXUlFlo91Tg2WpOkGARC1WS5S8t0/edit?usp=sharing), generated with kicad-footprint-generator")
 		(tags "capacitor")
-		(property "Reference" "CУ1"
+		(property "Reference" "CU1"
 			(at 0 -1.68 0)
 			(layer "F.SilkS")
