File: mcu_atmega_spi.kicad_sch (KiCad schematic)
At the start: 29 parts, among them J5 AVR ICSP, J6 Conn_01x01, J7 Conn_01x01, J8 Conn_01x01, J9 Conn_01x01, SW1 SW_Push, SW2 SW_Push, SW3 SW_Push, U5 ATmega328P-A, U6 CP2102N-A02-GQFN28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

Commit message: Force update local files
Parts:
- added H1, H2, H3, H4: MountingHole, MountingHole:MountingHole_3.2mm_M3, symbol Mechanical:MountingHole
- added J10: Conn_01x01, Connector_PinHeader_2.54mm:PinHeader_1x01_P2.54mm_Vertical, symbol Connector_Generic:Conn_01x01
- C1, C2, C23, C27, C28, C29, C3, C30, C31, C32: footprint Capacitor_THT:C_Disc_D5.0mm_W2.5mm_P5.00mm -> Capacitor_SMD:C_0805_2012Metric
- SW1, SW2, SW3: footprint Button_Switch_THT:SW_PUSH_6mm -> Button_Switch_SMD:SW_SPST_PTS645Sx43SMTR92
Connections:
- net PC3: now also J10.1 (Pin_1); no longer J9.1 (Pin_1), R15.2
- new net: J9.1 (Pin_1), R15.2

Commit message: done with lcsc
Parts:
- C1, C2, C23, C27, C28, C3, C31, C32: LCSC C1591 -> C1711
- C29, C30: LCSC (none) -> C472840
- FB3: value FerriteBead -> 600Ω @ 100MHz; LCSC C1015 -> C21519
- J5: LCSC C65114 -> (none)
- R15: LCSC (none) -> C2933324
- R18, R19, R21, R22, R23, R3: LCSC C25744 -> C543567
- SW1, SW2, SW3: LCSC C318884 -> C2834918
- U6: LCSC C1550553 -> C964632
- Y2: LCSC C13738 -> C7275095

Commit message: production
Parts:
- J10, J5, J6, J7, J8, J9: now not fitted

Commit message: .
Changed lines of the file:
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@@
 		(in_pos_files yes)
 		(dnp yes)
-		(fields_autoplaced yes)
 		(property "Reference" "C30"
-			(at 130.81 85.09 90)
+			(at 130.556 86.36 90)
 			(show_name no)
 			(do_not_autoplace no)
@@
 		)
 		(property "Value" "27pF"
-			(at 130.81 87.63 90)
+			(at 130.81 92.71 90)
 			(show_name no)
 			(do_not_autoplace no)
@@
 		(dnp no)
 		(property "Reference" "R19"
-			(at 119.38 105.41 90)
+			(at 119.38 108.458 90)
 			(show_name no)
 			(do_not_autoplace no)
@@
 		)
 		(property "Value" "10K"
-			(at 119.38 107.95 90)
+			(at 119.38 110.49 90)
 			(show_name no)
 			(do_not_autoplace no)
@@
 		(in_pos_files yes)
 		(dnp no)
-		(fields_autoplaced yes)
 		(property "Reference" "R18"
-			(at 120.65 99.0599 0)
+			(at 116.84 99.06 0)
 			(show_name no)
 			(do_not_autoplace no)
@@
 		)
 		(property "Value" "10K"
-			(at 120.65 101.5999 0)
-			(show_name no)
-			(do_not_autoplace no)
+			(at 117.094 100.584 0)
+			(show_name no)
+			(do_not_autoplace no)
