File: power_usb_battery_buck.kicad_sch (KiCad schematic)
At the start: 41 parts, among them J1 JST-XH 3-pin, J2 USB_C_Receptacle_USB2.0_16P, Q1 AO3400A, Q2 AO3400A, Q3 AO3400A, Q4 AO3400A, Q5 AO3400A, Q6 IRLML6244, Q7 IRLML6244, U1 HY2120-CB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

Commit message: Force update local files
Parts:
- C10, C16, C33, C34, C9: footprint Capacitor_THT:CP_Radial_D5.0mm_P2.00mm -> Capacitor_SMD:CP_Elec_5x5.4
- C11, C14, C15, C17, C18, C19, C8: footprint Capacitor_THT:C_Disc_D5.0mm_W2.5mm_P5.00mm -> Capacitor_SMD:C_0805_2012Metric
- D1: footprint LED_THT:LED_D5.0mm -> LED_SMD:LED_0805_2012Metric
- L1, L2: footprint Inductor_THT:L_Radial_D10.0mm_P5.00mm_Fastron_07M -> Inductor_SMD:L_10.4x10.4_H4.8
Changed lines of the file:
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@@
 			)
 		)
-		(property "Footprint" "Capacitor_THT:CP_Radial_D5.0mm_P2.00mm"
+		(property "Footprint" "Capacitor_SMD:CP_Elec_5x5.4"
 			(at 82.55 77.47 0)
 			(effects
@@
 			)
 		)
-		(property "Footprint" "Capacitor_THT:CP_Radial_D5.0mm_P2.00mm"
+		(property "Footprint" "Capacitor_SMD:CP_Elec_5x5.4"
 			(at 227.33 144.78 0)
 			(effects
@@
 			)
 		)
-		(property "Footprint" "Capacitor_THT:C_Disc_D5.0mm_W2.5mm_P5.00mm"
+		(property "Footprint" "Capacitor_SMD:C_0805_2012Metric"
 			(at 115.57 88.9 0)
 			(effects
@@
 			)
 		)
-		(property "Footprint" "Capacitor_THT:C_Disc_D5.0mm_W2.5mm_P5.00mm"
+		(property "Footprint" "Capacitor_SMD:C_0805_2012Metric"
 			(at 173.99 40.64 0)
 			(effects
@@
 			)
 		)
-		(property "Footprint" "Capacitor_THT:CP_Radial_D5.0mm_P2.00mm"
+		(property "Footprint" "Capacitor_SMD:CP_Elec_5x5.4"
 			(at 270.51 154.94 0)
 			(effects
@@
 			)
 		)
-		(property "Footprint" "Inductor_THT:L_Radial_D10.0mm_P5.00mm_Fastron_07M"
+		(property "Footprint" "Inductor_SMD:L_10.4x10.4_H4.8"
 			(at 270.51 142.24 0)
 			(effects
@@
 			)
 		)
-		(property "Footprint" "Capacitor_THT:C_Disc_D5.0mm_W2.5mm_P5.00mm"
+		(property "Footprint" "Capacitor_SMD:C_0805_2012Metric"
 			(at 82.55 72.39 0)
 			(effects
@@
 			)
 		)
-		(property "Footprint" "Capacitor_THT:C_Disc_D5.0mm_W2.5mm_P5.00mm"
+		(property "Footprint" "Capacitor_SMD:C_0805_2012Metric"
 			(at 107.95 106.68 0)
 			(effects
@@
 			)
 		)
-		(property "Footprint" "Capacitor_THT:C_Disc_D5.0mm_W2.5mm_P5.00mm"
+		(property "Footprint" "Capacitor_SMD:C_0805_2012Metric"
 			(at 154.94 40.64 0)
 			(effects
@@
 			)
 		)
-		(property "Footprint" "LED_THT:LED_D5.0mm"
+		(property "Footprint" "LED_SMD:LED_0805_2012Metric"
 			(at 153.67 153.67 90)
 			(effects
@@
 			)
 		)
-		(property "Footprint" "Capacitor_THT:CP_Radial_D5.0mm_P2.00mm"
+		(property "Footprint" "Capacitor_SMD:CP_Elec_5x5.4"
 			(at 222.25 58.42 0)
 			(effects
@@
 			)
 		)
-		(property "Footprint" "Inductor_THT:L_Radial_D10.0mm_P5.00mm_Fastron_07M"
+		(property "Footprint" "Inductor_SMD:L_10.4x10.4_H4.8"
 			(at 154.94 26.67 0)
 			(effects
@@
 			)
 		)
-		(property "Footprint" "Capacitor_THT:C_Disc_D5.0mm_W2.5mm_P5.00mm"
+		(property "Footprint" "Capacitor_SMD:C_0805_2012Metric"
 			(at 217.17 58.42 0)
 			(effects
@@
 			)
 		)
-		(property "Footprint" "Capacitor_THT:C_Disc_D5.0mm_W2.5mm_P5.00mm"
+		(property "Footprint" "Capacitor_SMD:C_0805_2012Metric"
 			(at 113.03 116.84 0)
 			(effects
@@
 			)
 		)
-		(property "Footprint" "Capacitor_THT:CP_Radial_D5.0mm_P2.00mm"
+		(property "Footprint" "Capacitor_SMD:CP_Elec_5x5.4"
 			(at 219.71 96.52 0)
 			(effects

Commit message: done with lcsc
Parts:
- C10: footprint Capacitor_SMD:CP_Elec_5x5.4 -> Capacitor_SMD:C_0805_2012Metric; LCSC C145095 -> C239256
- C11, C8: LCSC C1591 -> C1711
- C14, C15: LCSC C17250543 -> C53134
- C16: footprint Capacitor_SMD:CP_Elec_5x5.4 -> Capacitor_SMD:C_0805_2012Metric; LCSC C427012 -> C98195
- C17: LCSC C5128425 -> C1791
- C18: LCSC C21122 -> C1729
- C19: LCSC C1634 -> C2319426
- C33: footprint Capacitor_SMD:CP_Elec_5x5.4 -> Capacitor_SMD:C_0805_2012Metric; LCSC C17024 -> C98195
- C34: footprint Capacitor_SMD:CP_Elec_5x5.4 -> Capacitor_SMD:C_0805_2012Metric; LCSC C45783 -> C602037
- C9: footprint Capacitor_SMD:CP_Elec_5x5.4 -> Capacitor_SMD:C_0805_2012Metric; LCSC C2969873 -> C7469956
- D1: LCSC (none) -> C84260
- F1: LCSC C207023 -> C2840556
- J1: LCSC C161870 -> (none)
- J2: LCSC C132563 -> C2988369
- L1: value L -> 2.2µH; LCSC C1046 -> C10164
- L2: LCSC C1045 -> C19633496
- Q6, Q7: LCSC C143946 -> C5364311
- R1: LCSC C22944 -> C6460768
- R10: LCSC C25879 -> C441982
- R11: LCSC C4160698 -> C203741
- R12: LCSC C325870 -> C153307
- R13, R14: LCSC C2862317 -> C543567
- R2: LCSC C25741 -> C441992
- R4, R5: LCSC C25905 -> C491151
- R6: LCSC C11702 -> C844939
- R7, R8: LCSC (none) -> C308574
- R9: LCSC C2641913 -> C844598

Commit message: production
Parts:
- J1: now not fitted

Commit message: V2
Parts:
- C10: LCSC C239256 -> C602037
Changed lines of the file:
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@@
 			)
 		)
-		(property "LCSC" "C239256"
+		(property "LCSC" "C602037"
 			(at 222.25 58.42 0)
 			(hide yes)

Commit message: .
Changed lines of the file:
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@@
 	(wire
 		(pts
+			(xy 26.67 160.02) (xy 30.48 162.56)
+		)
+		(stroke
+			(width 0)
+			(type default)
+		)
+	)
+	(wire
+		(pts
 			(xy 53.34 160.02) (xy 90.17 160.02)
 		)
@@
 	)
 	(label "VBAT-"
-		(at 30.48 162.56 180)
+		(at 26.67 160.02 180)
 		(effects
 			(font
@@
 	(symbol
 		(lib_id "power:GND")
-		(at 139.7 38.1 270)
+		(at 139.7 38.1 0)
 		(unit 1)
 		(body_style 1)
@@
 		(dnp no)
 		(property "Reference" "#PWR020"
-			(at 133.35 38.1 0)
+			(at 139.7 44.45 0)
 			(hide yes)
 			(show_name no)
@@
 		)
 		(property "Value" "GND"
-			(at 144.018 38.608 90)
+			(at 144.018 38.354 0)
 			(show_name no)
 			(do_not_autoplace no)
